File: PCB Files/adapters/sanni_snes_shield/sanni_snes.kicad_pcb (KiCad board)
At the start: 2 copper layers, 59.5 x 90 mm, 9 parts, among them J1 SNES_EXP_CONN, J2 CLOCKGEN, SW1 CLK0, SW2 CLK1, U1 PIC12F629-ISN

Commit message: Add files via upload
Parts:
- removed Ref**: Val**, misc_footprints:ein1
